Commit message: almost kodu 3

File: src/my_r2d2/urdf/r2d2.xacro (robot description, xacro)
@@ -37,4 +37,11 @@
     <xacro:default_inertial mass="10"/>
   </link>
+  <link name="base_footprint">
+  </link>
+  <joint name="basetofootprint" type="fixed">
+    <parent link="base_link"/>
+    <child link="base_footprint"/>
+    <origin xyz="0 0 ${-((bodylen/2)+0.1+wheeldiam)}"/>
+  </joint>
   <xacro:macro name="wheel" params="prefix suffix reflect">
     <link name="${prefix}_${suffix}_wheel">

Commit message: Kodu 3

File: src/my_r2d2/urdf/r2d2.xacro (robot description, xacro)
@@ -40,7 +40,7 @@
   </link>
   <joint name="basetofootprint" type="fixed">
-    <parent link="base_link"/>
-    <child link="base_footprint"/>
-    <origin xyz="0 0 ${-((bodylen/2)+0.1+wheeldiam)}"/>
+    <parent link="base_footprint"/>
+    <child link="base_link"/>
+    <origin xyz="0 0 ${((bodylen/2)+0.1+wheeldiam)}"/>
   </joint>
   <xacro:macro name="wheel" params="prefix suffix reflect">

Commit message: kodu 4 done

File: src/my_r2d2/urdf/r2d2.xacro (robot description, xacro)
@@ -242,3 +242,10 @@
     <origin xyz="0.001 0 0.001"/>
   </joint>
+  <link name="eye">
+  </link>
+  <joint name="eyetolens" type="fixed">
+    <parent link="lense"/>
+    <child link="eye"/>
+    <origin xyz="0 0 0" rpy="-1.57075 0 -1.57075"/>
+  </joint>
 </robot>

Commit message: Kodu_6 Done

File: src/my_r2d2/urdf/r2d2.xacro (robot description, xacro)
@@ -247,5 +247,5 @@
     <parent link="lense"/>
     <child link="eye"/>
-    <origin xyz="0 0 0" rpy="-1.57075 0 -1.57075"/>
+    <origin xyz="0 0 0" rpy="${-(pi/2)} 0 ${-(pi/2)}"/>
   </joint>
 </robot>
